File: kicad/CoinboxV2.kicad_pcb (KiCad board)
At the start: 2 copper layers, 52.7 x 86.4 mm, 18 parts, among them J1 Conn_01x03, J2 Jack-DC, J3 Conn_01x03, Q2 2N7000

Commit message: PCB Rev 2.1
Signed-off-by: Patrick Pedersen <ctx.xda@gmail.com>
Parts:
- removed Q2: 2N7000, Package_TO_SOT_THT:TO-92_HandSolder
- J1: footprint Connector_JST:JST_XH_S3B-XH-A-1_1x03_P2.50mm_Horizontal -> Connector_Wire:SolderWire-0.1sqmm_1x03_P3.6mm_D0.4mm_OD1mm; moved to B.Cu
- moved J1 1.53 mm to (87.0, 134.9)
Connections:
- J2 pad 1: 5V -> GND
- J2 pad 2: GND -> 5V
- U2 pad 5: Net-(Q2-D) -> GND
- U3 pad 11: Net-(Q2-G) -> unconnected-(U3-GPIO35-Pad11)
Routing:
- net Net-(Q2-D): track 58.2 -> 0.00 mm
- net Net-(Q2-G): track 18.7 -> 0.00 mm
- net GND: track 39.2 -> 48.8 mm
- net SENS_3V3: track 16.9 -> 24.5 mm
- net /SENS_SIG: track 43.2 -> 40.0 mm
- net 5V: track 126.7 -> 129.2 mm
Other:
- board text added: "Coin Box Rev 2.1"
- board text removed: "Coin Box Rev 2.0"
