File: kicad/CoinboxV2.kicad_sch (KiCad schematic)
At the start: 14 parts, among them J1 Conn_01x03, J2 Jack-DC, J3 Conn_01x03, Q2 2N7000

Commit message: PCB Rev 2.1
Signed-off-by: Patrick Pedersen <ctx.xda@gmail.com>
Parts:
- removed Q2: 2N7000, Package_TO_SOT_THT:TO-92_Inline, symbol Transistor_FET:2N7000
- C1: value C -> 100n
- J1: footprint Connector_JST:JST_XH_S3B-XH-A-1_1x03_P2.50mm_Horizontal -> Connector_Wire:SolderWire-0.1sqmm_1x03_P3.6mm_D0.4mm_OD1mm
Connections:
- net 5V: now also J2.2; no longer J2.1
- net GND: now also J2.1, U2.5 (-/GND); no longer J2.2
- no-connect marks 26 -> 27
Other:
- note added: "Coin Box Revision 2.1"
- note removed: "Coin Box Revision 2.0"
- note removed: "The speaker stays muted via Q2 until the first coin is inserted. After detecting a coin, the system disables Wi-Fi (which is used for device configuration) and unmutes the speaker. This is done because Wi-Fi introduces noticeable noise on the DAC output. For more details, refer to the firmware source code."
Changed lines of the file:
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@@
 	(title_block
 		(title "Coin Box")
-		(date "2025-07-20")
-		(rev "2.0")
+		(date "2025-08-06")
+		(rev "2.1")
 		(company "TuDo Makerspace")
 	)
@@
 		)
 		(fill
-			(type outline)
+			(type color)
+			(color 0 0 0 0)
 		)
 	)
@@
 		)
 		(fill
-			(type outline)
+			(type color)
+			(color 0 0 0 0)
 		)
 	)
@@
 		)
 		(fill
-			(type outline)
+			(type color)
+			(color 0 0 0 0)
 		)
 	)
@@
 		)
 		(fill
-			(type outline)
+			(type color)
+			(color 0 0 0 0)
 		)
 	)
@@
 		)
 		(fill
-			(type outline)
+			(type color)
+			(color 0 0 0 0)
 		)
 	)
@@
 		)
 	)
-	(text "Coin Box Revision 2.0"
+	(text "Coin Box Revision 2.1"
 		(exclude_from_sim no)
 		(at 14.732 23.114 0)
@@
 		)
 	)
-	(text "The speaker stays muted via Q2 until\nthe first coin is inserted. After \ndetecting a coin, the system disables \nWi-Fi (which is used for device\nconfiguration) and unmutes the \nspeaker. This is done because Wi-Fi\nintroduces noticeable noise on the\nDAC output. For more details, refer\nto the firmware source code."
-		(exclude_from_sim no)
-		(at 154.686 128.27 0)
-		(effects
-			(font
-				(face "KiCad Font")
-				(size 1.27 1.27)
-				(thickness 0.1588)
-			)
-			(justify left)
-		)
-	)
 	(junction
 		(at 170.18 187.96)
@@
 	)
 	(no_connect
+		(at 87.63 109.22)
+	)
+	(no_connect
 		(at 129.54 109.22)
 	)
@@
 	(wire
 		(pts
-			(xy 87.63 109.22) (xy 104.14 109.22)
-		)
-		(stroke
-			(width 0)
-			(type default)
-		)
-	)
-	(wire
-		(pts
 			(xy 157.48 160.02) (xy 163.83 160.02)
 		)
@@
 	(wire
 		(pts
-			(xy 140.97 128.27) (xy 140.97 132.08)
+			(xy 140.97 115.57) (xy 140.97 119.38)
 		)
 		(stroke
@@
 	(wire
 		(pts
-			(xy 140.97 115.57) (xy 140.97 118.11)
-		)
-		(stroke
-			(width 0)
-			(type default)
-		)
-	)
-	(wire
-		(pts
 			(xy 132.08 176.53) (xy 144.78 176.53)
 		)
@@
 	(wire
 		(pts
-			(xy 133.35 123.19) (xy 104.14 123.19)
-		)
-		(stroke
-			(width 0)
-			(type default)
-		)
-	)
-	(wire
-		(pts
 			(xy 55.88 78.74) (xy 55.88 83.82)
 		)
@@
 		(pts
 			(xy 30.48 86.36) (xy 41.91 86.36)
-		)
-		(stroke
-			(width 0)
-			(type default)
-		)
-	)
-	(wire
-		(pts
-			(xy 104.14 123.19) (xy 104.14 109.22)
 		)
 		(stroke
@@
 	)
 	(symbol
-		(lib_id "Transistor_FET:2N7000")
-		(at 138.43 123.19 0)
-		(unit 1)
-		(exclude_from_sim no)
-		(in_bom yes)
-		(on_board yes)
-		(dnp no)
-		(fields_autoplaced yes)
-		(property "Reference" "Q2"
-			(at 144.78 121.9199 0)
-			(effects
-				(font
-					(size 1.27 1.27)
-				)
-				(justify left)
-			)
-		)
-		(property "Value" "2N7000"
-			(at 144.78 124.4599 0)
-			(effects
-				(font
-					(size 1.27 1.27)
-				)
-				(justify left)
-			)
-		)
-		(property "Footprint" "Package_TO_SOT_THT:TO-92_Inline"
-			(at 143.51 125.095 0)
-			(effects
-				(font
-					(size 1.27 1.27)
-					(italic yes)
-				)
-				(justify left)
-				(hide yes)
-			)
-		)
-		(property "Datasheet" "https://www.vishay.com/docs/70226/70226.pdf"
-			(at 143.51 127 0)
-			(effects
-				(font
-					(size 1.27 1.27)
-				)
-				(justify left)
-				(hide yes)
-			)
-		)
-		(property "Description" "0.2A Id, 200V Vds, N-Channel MOSFET, 2.6V Logic Level, TO-92"
-			(at 138.43 123.19 0)
-			(effects
-				(font
-					(size 1.27 1.27)
-				)
-				(hide yes)
-			)
-		)
-		(pin "1"
-		)
-		(pin "3"
-		)
-		(pin "2"
-		)
-		(instances
-			(project ""
-				(path "/9253c832-1fb2-4ef4-b559-448e617d6971"
-					(reference "Q2")
-					(unit 1)
-				)
-			)
-		)
-	)
-	(symbol
 		(lib_id "power:VCC")
 		(at 41.91 78.74 0)
@@
 	(symbol
 		(lib_id "power:GND")
-		(at 140.97 132.08 0)
+		(at 140.97 119.38 0)
 		(unit 1)
 		(exclude_from_sim no)
@@
 		(dnp no)
 		(property "Reference" "#PWR01"
-			(at 140.97 138.43 0)
+			(at 140.97 125.73 0)
 			(effects
 				(font
@@
 		)
 		(property "Value" "GND"
-			(at 140.97 137.16 0)
+			(at 140.97 124.46 0)
 			(effects
 				(font
@@
 		)
 		(property "Footprint" ""
-			(at 140.97 132.08 0)
+			(at 140.97 119.38 0)
 			(effects
 				(font
@@
 		)
 		(property "Datasheet" ""
-			(at 140.97 132.08 0)
+			(at 140.97 119.38 0)
 			(effects
 				(font
@@
 		)
 		(property "Description" "Power symbol creates a global label with name \"GND\" , ground"
-			(at 140.97 132.08 0)
+			(at 140.97 119.38 0)
 			(effects
 				(font
@@
 			)
 		)
-		(property "Value" "C"
+		(property "Value" "100n"
 			(at 185.42 175.2599 0)
 			(effects
@@
 		(on_board yes)
 		(dnp no)
-		(fields_autoplaced yes)
 		(property "Reference" "J2"
 			(at 22.86 74.93 0)
@@
 			)
 		)
-		(property "Footprint" "Connector_JST:JST_XH_S3B-XH-A-1_1x03_P2.50mm_Horizontal"
+		(property "Footprint" "Connector_Wire:SolderWire-0.1sqmm_1x03_P3.6mm_D0.4mm_OD1mm"
 			(at 127 173.99 0)
 			(effects
